Commit message: Add sensor frames and TF2 robot transforms

File: src/robot_description/urdf/my_robot.urdf (robot description, URDF)
Before this commit: robot my_robot, 4 links, 3 joints
Links:
- added link camera_link; visual box size=0.04 0.08 0.04
- added link lidar_link; visual cylinder length=0.05 radius=0.04
Joints:
- added joint camera_joint: type fixed, parent base_link, child camera_link, origin xyz=0.18 0 0.12 rpy=0 0 0
- added joint lidar_joint: type fixed, parent base_link, child lidar_link, origin xyz=0.10 0 0.10 rpy=0 0 0

File: src/robot_description/urdf/my_robot.urdf.xacro (robot description, xacro)
@@ -49,3 +49,27 @@
     <origin xyz="-0.15 0 -0.04" rpy="0 0 0"/>
   </joint>
+  <link name="lidar_link">
+    <visual>
+      <geometry>
+        <cylinder radius="0.04" length="0.05"/>
+      </geometry>
+    </visual>
+  </link>
+  <joint name="lidar_joint" type="fixed">
+    <parent link="base_link"/>
+    <child link="lidar_link"/>
+    <origin xyz="0.10 0 0.10" rpy="0 0 0"/>
+  </joint>
+  <link name="camera_link">
+    <visual>
+      <geometry>
+        <box size="0.04 0.08 0.04"/>
+      </geometry>
+    </visual>
+  </link>
+  <joint name="camera_joint" type="fixed">
+    <parent link="base_link"/>
+    <child link="camera_link"/>
+    <origin xyz="0.18 0 0.12" rpy="0 0 0"/>
+  </joint>
 </robot>
